Commit message: feat: grand transfer (fix_sim)

File: overlord100_simulation/description/overlord100.urdf.xacro (robot description, xacro)
@@ -1,14 +1,457 @@
 <?xml version="1.0"?>
-<!-- Basic differential drive mobile base -->
-<robot xmlns:xacro="http://www.ros.org/wiki/xacro" name="overlord100_simulation_test">
-  <xacro:arg name="prefix" default="" />
-  <xacro:arg name="use_mock_hardware" default="false" />
-  <xacro:include filename="$(find overlord100_simulation)/urdf/overlord100_description.urdf.xacro" />
-  <!-- Import Rviz colors -->
-  <!-- <xacro:include filename="$(find ros2_control_demo_description)/diffbot/urdf/diffbot.materials.xacro" /> -->
-  <!-- Import overlord100 ros2_control description -->
-  <xacro:include filename="$(find overlord100_simulation)/ros2_control/overlord100.ros2_control.xacro" />
-  <xacro:overlord100 prefix="$(arg prefix)" />
-  <xacro:overlord100_ros2_control
-    name="Overlord100" prefix="$(arg prefix)" use_mock_hardware="$(arg use_mock_hardware)"/>
+<robot xmlns:xacro="http://ros.org/wiki/xacro" name="overlord100">
+    <!-- Include Gazebo Parameters -->
+    <xacro:include filename="$(find overlord100_simulation)/description/overlord100_gazebo.xacro" />
+    <!-- Include ROS2 Control -->
+    <xacro:include filename="$(find overlord100_simulation)/description/overlord100_control.xacro" />
+    <link name="base_footprint"/>
+    <link name="base_link">
+        <visual>
+            <origin rpy="0 0 -1.57075" xyz="0 0 -0.20" />
+            <geometry>
+                <mesh filename="package://overlord100_simulation/models/base.dae"/>
+            </geometry>
+        </visual>
+        <inertial>
+            <mass value="60.5" />
+            <inertia ixx="0.45375" ixy="0.0" ixz="0.0" iyy="2.263304" iyz="0.0" izz="2.716954" />
+        </inertial>
+        <collision>
+            <geometry>
+                <box size="0.93 0.67 0.2" />
+            </geometry>
+        </collision>
+    </link>
+    <joint name="base_joint" type="fixed">
+        <parent link="base_footprint" />
+        <child link="base_link" />
+        <origin rpy="0 0 0" xyz="0 0 0.20" />
+    </joint>
+    <!-- wheels -->
+    <link name="left_wheel">
+        <visual>
+            <origin rpy="0 0 -1.57075" xyz="0 0 -0.0655" />
+            <geometry>
+                <mesh filename = "package://overlord100_simulation/models/left_wheel.dae"  />
+            </geometry>
+        </visual>
+        <inertial>
+            <mass value="1" />
+            <inertia ixx="0.0175" ixy="0.0" ixz="0.0" iyy="0.0175" iyz="0.0" izz="0.02" />
+        </inertial>
+        <collision>
+            <origin rpy="1.57075 0 0" xyz="0 0 0" />
+            <geometry>
+                <cylinder radius = "0.07" length = "0.06" />
+            </geometry>
+        </collision>
+    </link>
+    <joint name="base_link_to_left_wheel" type="continuous">
+        <axis xyz="0 1 0" />
+        <limit effort="1000.0" lower="-1.79769e+308" upper="1.79769e+308" velocity="100.0" />
+        <parent link="base_link" />
+        <child link="left_wheel" />
+        <origin rpy="0 0 0" xyz="-0.045 0.33 -0.15" />
+    </joint>
+    <link name="right_wheel">
+        <visual>
+            <origin rpy="0 0 -1.57075" xyz="0 0 -0.0655" />
+            <geometry>
+                <mesh filename = "package://overlord100_simulation/models/right_wheel.dae"/>
+            </geometry>
+        </visual>
+        <inertial>
+            <mass value="1" />
+            <inertia ixx="0.0175" ixy="0.0" ixz="0.0" iyy="0.0175" iyz="0.0" izz="0.02" />
+        </inertial>
+        <collision>
+            <origin rpy="1.57075 0 0" xyz="0 0 0" />
+            <geometry>
+                <cylinder radius = "0.07" length = "0.06" />
+            </geometry>
+        </collision>
+    </link>
+    <joint name="base_link_to_right_wheel" type="continuous">
+        <axis xyz="0 1 0" />
+        <limit effort="1000.0" lower="-1.79769e+308" upper="1.79769e+308" velocity="100.0" />
+        <parent link="base_link" />
+        <child link="right_wheel" />
+        <origin rpy="0 0 0" xyz="-0.045 -0.33 -0.15" />
+    </joint>
+    <link name="front_left_dummy_wheel">
+        <visual>
+        <origin rpy="0 0 -1.57075" xyz=" 0 0 -0.07" />
+            <geometry>
+                <mesh filename = "package://overlord100_simulation/models/front_left_wheel.dae" />
+                <!-- <sphere radius="0.2" /> -->
+            </geometry>
+        </visual>
+        <inertial>
+            <mass value="1" />
+            <inertia ixx="0.016" ixy="0.0" ixz="0.0" iyy="0.016" iyz="0.0" izz="0.016" />
+        </inertial>
+        <collision>
+            <geometry>
+                <sphere radius= "0.07" />
+            </geometry>
+        </collision>
+    </link>
+    <joint name="base_link_to_front_left_dummy_wheel" type="fixed">
+        <parent link="base_link" />
+            <child link="front_left_dummy_wheel" />
+        <origin rpy="0 0 0" xyz="0.40 -0.23 -0.15" />
+    </joint>
+    <link name="front_right_dummy_wheel">
+        <visual>
+            <origin rpy="0 0 -1.57075" xyz=" 0 0 -0.07" />
+            <geometry>
+                <mesh filename = "package://overlord100_simulation/models/front_right_wheel.dae" />
+                <!-- <sphere radius="0.2" /> -->
+            </geometry>
+        </visual>
+        <inertial>
+            <mass value="1" />
+            <inertia ixx="0.016" ixy="0.0" ixz="0.0" iyy="0.016" iyz="0.0" izz="0.016" />
+        </inertial>
+        <collision>
+            <geometry>
+                <sphere radius= "0.07" />
+            </geometry>
+        </collision>
+    </link>
+    <joint name="base_link_to_front_right_dummy_wheel" type="fixed">
+        <parent link="base_link" />
+        <child link="front_right_dummy_wheel" />
+        <origin rpy="0 0 0" xyz="0.40 0.23 -0.15" />
+    </joint>
+    <link name="back_right_dummy_wheel">
+        <visual>
+            <origin rpy="0 0 -1.57075" xyz=" 0 0 -0.07" />
+            <geometry>
+                <mesh filename = "package://overlord100_simulation/models/back_right_wheel.dae"  />
+                <!-- <sphere radius="0.2" /> -->
+            </geometry>
+        </visual>
+        <inertial>
+            <mass value="1" />
+            <inertia ixx="0.016" ixy="0.0" ixz="0.0" iyy="0.016" iyz="0.0" izz="0.016" />
+        </inertial>
+        <collision>
+            <geometry>
+                <sphere radius= "0.07" />
+            </geometry>
+        </collision>
+    </link>
+    <joint name="base_link_to_back_right_dummy_wheel" type="fixed">
+        <parent link="base_link" />
+        <child link="back_right_dummy_wheel" />
+        <origin rpy="0 0 0" xyz="-0.42  0.27 -0.15" />
+    </joint>
+    <link name="back_left_dummy_wheel">
+        <visual>
+            <origin rpy="0 0 -1.57075" xyz=" 0 0 -0.07" />
+            <geometry>
+                <mesh filename = "package://overlord100_simulation/models/back_left_wheel.dae"  />
+                <!-- <sphere radius="0.2" /> -->
+            </geometry>
+        </visual>
+        <collision>
+            <geometry>
+                <sphere radius= "0.07" />
+            </geometry>
+        </collision>
+        <inertial>
+            <mass value="1" />
+            <inertia ixx="0.016" ixy="0.0" ixz="0.0" iyy="0.016" iyz="0.0" izz="0.016" />
+        </inertial>
+    </link>
+    <joint name="base_link_to_back_left_dummy_wheel" type="fixed">
+        <parent link="base_link" />
+        <child link="back_left_dummy_wheel" />
+        <origin rpy="0 0 0" xyz="-0.42 -0.27 -0.15" />
+    </joint>
+    <!-- lidars -->
+    <link name="lidar_front">
+        <visual>
+            <geometry>
+                <mesh filename = "package://overlord100_simulation/models/front_lidar.dae"  />
+                <!-- <cylinder length="0.06" radius="0.09" /> -->
+            </geometry>
+        </visual>
+        <inertial>
+            <mass value="0.1" />
+            <inertia ixx="0.000158" ixy="0.0" ixz="0.0" iyy="0.000158" iyz="0.0" izz="0.00018" />
+        </inertial>
+        <collision>
+            <geometry>
+                <box size = "0.061 0.041 0.055" />
+            </geometry>
+        </collision>
+    </link>
+    <joint name="base_link_to_lidar_front" type="fixed">
+        <parent link="base_link" />
+        <child link="lidar_front" />
+        <origin rpy="0 0 0" xyz="0.43 0.26 0" />
+    </joint>
+    <link name="lidar_back">
+        <visual>
+            <geometry>
+                <mesh filename = "package://overlord100_simulation/models/back_lidar.dae"  />
+                <!-- <cylinder length="0.06" radius="0.09" /> -->
+            </geometry>
+        </visual>
+        <inertial>
+            <mass value="0.1" />
+            <inertia ixx="0.000158" ixy="0.0" ixz="0.0" iyy="0.000158" iyz="0.0" izz="0.00018" />
+        </inertial>
+        <collision>
+            <geometry>
+                <box size = "0.061 0.041 0.055" />
+            </geometry>
+        </collision>
+    </link>
+    <joint name="base_link_to_lidar_back" type="fixed">
+        <parent link="base_link" />
+        <child link="lidar_back" />
+        <origin rpy="0 0 0" xyz="-0.42 -0.26 0" />
+    </joint>
+    <!-- camera -->
+    <link name="realsense">
+        <visual>
+            <origin rpy="0 0 -1.57075" xyz="0 0 0"/>
+            <geometry>
+                <mesh filename = "package://overlord100_simulation/models/realsense.dae"  />
+                <!-- <cylinder length="0.06" radius="0.09" /> -->
+            </geometry>
+        </visual>
+        <inertial>
+            <mass value="0.1" />
+            <inertia ixx="0.000158" ixy="0.0" ixz="0.0" iyy="0.000158" iyz="0.0" izz="0.00018" />
+        </inertial>
+        <collision>
+            <geometry>
+                <box size = "0.061 0.041 0.055" />
+            </geometry>
+        </collision>
+    </link>
+    <joint name = "base_link_to_realsense" type = "fixed">
+        <parent link="base_link" />
+        <child link="realsense" />
+        <origin xyz = "0.4745 0 -0.0332"/>
+    </joint>
+    <!-- sonars -->
+    <link name="sonar1">
+        <visual>
+            <origin rpy="0 0 -1.57075" xyz="0 0 0"/>
+            <geometry>
+                <mesh filename = "package://overlord100_simulation/models/sonar1.dae"/>
+                <!-- <cylinder length="0.06" radius="0.09" /> -->
+            </geometry>
+        </visual>
+        <inertial>
+            <mass value="0.1" />
+            <inertia ixx="0.000158" ixy="0.0" ixz="0.0" iyy="0.000158" iyz="0.0" izz="0.00018" />
+        </inertial>
+        <collision>
+            <geometry>
+                <box size = "0.061 0.041 0.055" />
+            </geometry>
+        </collision>
+    </link>
+    <joint name = "base_link_to_sonar1" type = "fixed">
+        <parent link="base_link" />
+        <child link="sonar1" />
+        <origin xyz = "0.45 0.138 -0.032" rpy = "0 0 0"/>
+    </joint>
+    <link name="sonar2">
+        <visual>
+            <origin rpy="0 0 -1.57075" xyz="0 0 0"/>
+            <geometry>
+                <mesh filename = "package://overlord100_simulation/models/sonar2.dae"  />
+                <!-- <cylinder length="0.06" radius="0.09" /> -->
+            </geometry>
+        </visual>
+        <inertial>
+            <mass value="0.1" />
+            <inertia ixx="0.000158" ixy="0.0" ixz="0.0" iyy="0.000158" iyz="0.0" izz="0.00018" />
+        </inertial>
+        <collision>
+            <geometry>
+                <box size = "0.061 0.041 0.055" />
+            </geometry>
+        </collision>
+    </link>
+    <joint name = "base_link_to_sonar2" type = "fixed">
+        <parent link="base_link" />
+        <child link="sonar2" />
+        <origin xyz = " 0.45 -0.138 -0.032" rpy = "0 0 0"/>
+    </joint>
+    <link name="sonar3">
+        <visual>
+            <origin rpy="0 0.5 1.57075" xyz="0 0 0"/>
+            <geometry>
+                <mesh filename = "package://overlord100_simulation/models/sonar3.dae"  />
+                <!-- <cylinder length="0.06" radius="0.09" /> -->
+            </geometry>
+        </visual>
+        <inertial>
+            <mass value="0.1" />
+            <inertia ixx="0.000158" ixy="0.0" ixz="0.0" iyy="0.000158" iyz="0.0" izz="0.00018" />
+        </inertial>
+        <collision>
+            <geometry>
+                <box size = "0.061 0.041 0.055" />
+            </geometry>
+        </collision>
+    </link>
+    <joint name = "base_link_to_sonar3" type = "fixed">
+        <parent link="base_link" />
+        <child link="sonar3" />
+        <origin xyz = "0.24 -0.3 -0.032" rpy = "0.5 0 0"/>
+    </joint>
+    <link name="sonar4">
+        <visual>
+            <origin rpy="0 0.5 1.57075" xyz="0 0 0"/>
+            <geometry>
+                <mesh filename = "package://overlord100_simulation/models/sonar4.dae"  />
+                <!-- <cylinder length="0.06" radius="0.09" /> -->
+            </geometry>
+        </visual>
+        <inertial>
+            <mass value="0.1" />
+            <inertia ixx="0.000158" ixy="0.0" ixz="0.0" iyy="0.000158" iyz="0.0" izz="0.00018" />
+        </inertial>
+        <collision>
+            <geometry>
+                <box size = "0.061 0.041 0.055" />
+            </geometry>
+        </collision>
+    </link>
+    <joint name = "base_link_to_sonar4" type = "fixed">
+        <parent link="base_link" />
+        <child link="sonar4" />
+        <origin xyz = "-0.23 -0.3 -0.032" rpy = "0.5 0 0"/>
+    </joint>
+    <link name="sonar5">
+        <visual>
+            <origin rpy="0 0 1.57075" xyz="0 0 0"/>
+            <geometry>
+                <mesh filename = "package://overlord100_simulation/models/sonar5.dae"  />
+                <!-- <cylinder length="0.06" radius="0.09" /> -->
+            </geometry>
+        </visual>
+        <inertial>
+            <mass value="0.1" />
+            <inertia ixx="0.000158" ixy="0.0" ixz="0.0" iyy="0.000158" iyz="0.0" izz="0.00018" />
+        </inertial>
+        <collision>
+            <geometry>
+                <box size = "0.061 0.041 0.055" />
+            </geometry>
+        </collision>
+    </link>
+    <joint name = "base_link_to_sonar5" type = "fixed">
+        <parent link="base_link" />
+        <child link="sonar5" />
+        <origin xyz = "-0.45 -0.138 -0.032" rpy = "0 0 -3.1415"/>
+    </joint>
+    <link name="sonar6">
+        <visual>
+            <origin rpy="0 0 1.57075" xyz="0 0 0"/>
+            <geometry>
+                <mesh filename = "package://overlord100_simulation/models/sonar6.dae"  />
+                <!-- <cylinder length="0.06" radius="0.09" /> -->
+            </geometry>
+        </visual>
+        <inertial>
+            <mass value="0.1" />
+            <inertia ixx="0.000158" ixy="0.0" ixz="0.0" iyy="0.000158" iyz="0.0" izz="0.00018" />
+        </inertial>
+        <collision>
+            <geometry>
+                <box size = "0.061 0.041 0.055" />
+            </geometry>
+        </collision>
+    </link>
+    <joint name = "base_link_to_sonar6" type = "fixed">
+        <parent link="base_link" />
+        <child link="sonar6" />
+        <origin xyz = "-0.45 0.138 -0.032" rpy = "0 0 -3.1415"/>
+    </joint>
+    <link name="sonar7">
+        <visual>
+            <origin rpy="0 -0.5 0" xyz="0 0 0"/>
+            <geometry>
+                <mesh filename = "package://overlord100_simulation/models/sonar7.dae"  />
+                <!-- <cylinder length="0.06" radius="0.09" /> -->
+            </geometry>
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
Commit message: fix: /cmd_vel topic changed

File: overlord100_simulation/description/overlord100.urdf.xacro (robot description, xacro)
@@ -5,5 +5,4 @@
     <!-- Include ROS2 Control -->
     <xacro:include filename="$(find overlord100_simulation)/description/overlord100_control.xacro" />
-    <link name="base_footprint"/>
     <link name="base_link">
         <visual>
@@ -23,9 +22,4 @@
         </collision>
     </link>
-    <joint name="base_joint" type="fixed">
-        <parent link="base_footprint" />
-        <child link="base_link" />
-        <origin rpy="0 0 0" xyz="0 0 0.20" />
-    </joint>
     <!-- wheels -->
     <link name="left_wheel">
