Commit message: Changed wheel_radius and wheel_separarion and added IDE configs to .gitignor

File: navigation/iros_mobile_platform_description/description/iros_mobile_platform_description.urdf.xacro (robot description, xacro)
@@ -46,5 +46,5 @@
         <origin rpy="0 1.57075 0" xyz="0 0 0" />
         <geometry>
-          <cylinder radius="0.07" length="0.06" />
+          <cylinder radius="0.126" length="0.06" />
         </geometry>
       </collision>
@@ -55,5 +55,5 @@
       <parent link="chassis" />
       <child link="left_wheel" />
-      <origin rpy="0 0 3.14" xyz="-0.33 -0.045 -0.15" />
+      <origin rpy="0 0 3.14" xyz="-0.31 -0.045 -0.15" />
     </joint>
     <link name="lidar_front">
@@ -115,5 +115,5 @@
         <origin rpy="0 1.57075 0" xyz="0 0 0" />
         <geometry>
-          <cylinder radius="0.07" length="0.06" />
+          <cylinder radius="0.126" length="0.06" />
         </geometry>
       </collision>
@@ -124,5 +124,5 @@
       <parent link="chassis" />
       <child link="right_wheel" />
-      <origin rpy="0 0 3.14" xyz="0.33 -0.045 -0.15" />
+      <origin rpy="0 0 3.14" xyz="0.31 -0.045 -0.15" />
     </joint>
     <link name="front_left_dummy_wheel">
@@ -140,5 +140,5 @@
       <collision>
         <geometry>
-          <sphere radius="0.07" />
+          <sphere radius="0.126" />
         </geometry>
       </collision>
@@ -163,5 +163,5 @@
       <collision>
         <geometry>
-          <sphere radius="0.07" />
+          <sphere radius="0.126" />
         </geometry>
       </collision>
@@ -186,5 +186,5 @@
       <collision>
         <geometry>
-          <sphere radius="0.07" />
+          <sphere radius="0.126" />
         </geometry>
       </collision>
@@ -205,5 +205,5 @@
       <collision>
         <geometry>
-          <sphere radius="0.07" />
+          <sphere radius="0.126" />
         </geometry>
       </collision>
@@ -274,6 +274,6 @@
         <right_joint>chassis_to_right_wheel</right_joint>
         <!-- kinematics -->
-        <wheel_separation>0.34</wheel_separation>
-        <wheel_diameter>0.14</wheel_diameter>
+        <wheel_separation>0.62</wheel_separation>
+        <wheel_diameter>0.252</wheel_diameter>
         <!-- limits -->
         <max_wheel_torque>20</max_wheel_torque>

Commit message: fix(kinematics): correct wheel size calculation (use radius instead of diameter)

File: navigation/iros_mobile_platform_description/description/iros_mobile_platform_description.urdf.xacro (robot description, xacro)
@@ -46,5 +46,5 @@
         <origin rpy="0 1.57075 0" xyz="0 0 0" />
         <geometry>
-          <cylinder radius="0.126" length="0.06" />
+          <cylinder radius="0.063" length="0.06" />
         </geometry>
       </collision>
@@ -115,5 +115,5 @@
         <origin rpy="0 1.57075 0" xyz="0 0 0" />
         <geometry>
-          <cylinder radius="0.126" length="0.06" />
+          <cylinder radius="0.063" length="0.06" />
         </geometry>
       </collision>
@@ -140,5 +140,5 @@
       <collision>
         <geometry>
-          <sphere radius="0.126" />
+          <sphere radius="0.063" />
         </geometry>
       </collision>
@@ -163,5 +163,5 @@
       <collision>
         <geometry>
-          <sphere radius="0.126" />
+          <sphere radius="0.063" />
         </geometry>
       </collision>
@@ -205,5 +205,5 @@
       <collision>
         <geometry>
-          <sphere radius="0.126" />
+          <sphere radius="0.063" />
         </geometry>
       </collision>
@@ -275,5 +275,5 @@
         <!-- kinematics -->
         <wheel_separation>0.62</wheel_separation>
-        <wheel_diameter>0.252</wheel_diameter>
+        <wheel_diameter>0.126</wheel_diameter>
         <!-- limits -->
         <max_wheel_torque>20</max_wheel_torque>

Commit message: feat(everything): fix everything

File: navigation/iros_mobile_platform_description/description/iros_mobile_platform_description.urdf.xacro (robot description, xacro)
@@ -2,16 +2,9 @@
 <robot xmlns:xacro="http://www.ros.org/wiki/xacro">
   <xacro:macro name="iros_mobile_platform" params="prefix">
-    <link name="chassis1">
-      <visual>
-        <origin rpy="0 0 0" xyz="0 0 0" />
-        <!-- <geometry>
-        <mesh filename = "model://base.dae"/>
-      </geometry> -->
-      </visual>
-    </link>
-    <joint name="chassis1_2_chassis" type="fixed">
-      <parent link="chassis" />
-      <child link="chassis1" />
-      <origin rpy="0 0 1.57" xyz="0 0 0" />
+    <link name="base_link" />
+    <joint name="base_link_to_chassis" type="fixed">
+      <parent link="base_link" />
+      <child link="chassis" />
+      <origin rpy="0 0 -1.57079632679" xyz="0 0 0" />
     </joint>
     <link name="chassis">
@@ -77,5 +70,5 @@
       <parent link="chassis" />
       <child link="lidar_front" />
-      <origin rpy="0 0 0" xyz="0.26 0.43 0.01" />
+      <origin rpy="0 0 1.57079632679" xyz="0.26 0.43 0.01" />
     </joint>
     <link name="lidar_back">
@@ -99,5 +92,5 @@
       <parent link="chassis" />
       <child link="lidar_back" />
-      <origin rpy="0 0 0" xyz="-0.26 -0.42 0.01" />
+      <origin rpy="0 0 -1.57079632679" xyz="-0.26 -0.42 0.01" />
     </joint>
     <link name="right_wheel">
@@ -284,5 +277,5 @@
         <publish_wheel_tf>true</publish_wheel_tf>
         <odometry_frame>odom</odometry_frame>
-        <robot_base_frame>chassis</robot_base_frame>
+        <robot_base_frame>base_link</robot_base_frame>
       </plugin>
     </gazebo>
@@ -298,5 +291,5 @@
         <odom_topic>/odom</odom_topic>
         <odom_frame>odom</odom_frame>
-        <robot_base_frame>chassis</robot_base_frame>
+        <robot_base_frame>base_link</robot_base_frame>
         <tf_topic>/odom/tf</tf_topic>
       </plugin>

Commit message: fix(navigation): align URDF and scan merger geometry, add imu_link

File: navigation/iros_mobile_platform_description/description/iros_mobile_platform_description.urdf.xacro (robot description, xacro)
@@ -10,5 +10,5 @@
     <link name="chassis">
       <visual>
-        <origin rpy="0 0 0" xyz="0 0 -0.20" />
+        <origin rpy="0 0 3.14159265359" xyz="0 0 -0.20" />
         <geometry>
           <mesh filename="model://base.dae" />
@@ -25,4 +25,10 @@
       </collision>
     </link>
+    <link name="imu_link" />
+    <joint name="chassis_to_imu" type="fixed">
+      <parent link="chassis" />
+      <child link="imu_link" />
+      <origin rpy="0 0 0" xyz="0 0 0" />
+    </joint>
     <link name="left_wheel">
       <visual>
@@ -70,5 +76,5 @@
       <parent link="chassis" />
       <child link="lidar_front" />
-      <origin rpy="0 0 1.57079632679" xyz="0.26 0.43 0.01" />
+      <origin rpy="0 0 3.14159265359" xyz="0.26 0.43 0.01" />
     </joint>
     <link name="lidar_back">
@@ -92,5 +98,5 @@
       <parent link="chassis" />
       <child link="lidar_back" />
-      <origin rpy="0 0 -1.57079632679" xyz="-0.26 -0.42 0.01" />
+      <origin rpy="0 0 0" xyz="-0.26 -0.42 0.01" />
     </joint>
     <link name="right_wheel">

Commit message: fix(navigation): tune nav2 tolerances and calibrate wheel geometry to 130mm

File: navigation/iros_mobile_platform_description/description/iros_mobile_platform_description.urdf.xacro (robot description, xacro)
@@ -45,5 +45,5 @@
         <origin rpy="0 1.57075 0" xyz="0 0 0" />
         <geometry>
-          <cylinder radius="0.063" length="0.06" />
+          <cylinder radius="0.065" length="0.06" />
         </geometry>
       </collision>
@@ -114,5 +114,5 @@
         <origin rpy="0 1.57075 0" xyz="0 0 0" />
         <geometry>
-          <cylinder radius="0.063" length="0.06" />
+          <cylinder radius="0.065" length="0.06" />
         </geometry>
       </collision>
@@ -139,5 +139,5 @@
       <collision>
         <geometry>
-          <sphere radius="0.063" />
+          <sphere radius="0.065" />
         </geometry>
       </collision>
@@ -162,5 +162,5 @@
       <collision>
         <geometry>
-          <sphere radius="0.063" />
+          <sphere radius="0.065" />
         </geometry>
       </collision>
@@ -185,5 +185,5 @@
       <collision>
         <geometry>
-          <sphere radius="0.126" />
+          <sphere radius="0.130" />
         </geometry>
       </collision>
@@ -204,5 +204,5 @@
       <collision>
         <geometry>
-          <sphere radius="0.063" />
+          <sphere radius="0.065" />
         </geometry>
       </collision>
@@ -274,5 +274,5 @@
         <!-- kinematics -->
         <wheel_separation>0.62</wheel_separation>
-        <wheel_diameter>0.126</wheel_diameter>
+        <wheel_diameter>0.130</wheel_diameter>
         <!-- limits -->
         <max_wheel_torque>20</max_wheel_torque>

Commit message: Added corrections from dev branch

File: navigation/iros_mobile_platform_description/description/iros_mobile_platform_description.urdf.xacro (robot description, xacro)
@@ -2,20 +2,13 @@
 <robot xmlns:xacro="http://www.ros.org/wiki/xacro">
   <xacro:macro name="iros_mobile_platform" params="prefix">
-    <link name="chassis1">
-      <visual>
-        <origin rpy="0 0 0" xyz="0 0 0" />
-        <!-- <geometry>
-        <mesh filename = "model://base.dae"/>
-      </geometry> -->
-      </visual>
-    </link>
-    <joint name="chassis1_2_chassis" type="fixed">
-      <parent link="chassis" />
-      <child link="chassis1" />
-      <origin rpy="0 0 1.57" xyz="0 0 0" />
+    <link name="base_link" />
+    <joint name="base_link_to_chassis" type="fixed">
+      <parent link="base_link" />
+      <child link="chassis" />
+      <origin rpy="0 0 -1.57079632679" xyz="0 0 0" />
     </joint>
     <link name="chassis">
       <visual>
-        <origin rpy="0 0 0" xyz="0 0 -0.20" />
+        <origin rpy="0 0 3.14159265359" xyz="0 0 -0.20" />
         <geometry>
           <mesh filename="model://base.dae" />
@@ -32,4 +25,10 @@
       </collision>
     </link>
+    <link name="imu_link" />
+    <joint name="chassis_to_imu" type="fixed">
+      <parent link="chassis" />
+      <child link="imu_link" />
+      <origin rpy="0 0 0" xyz="0 0 0" />
+    </joint>
     <link name="left_wheel">
       <visual>
@@ -46,5 +45,5 @@
         <origin rpy="0 1.57075 0" xyz="0 0 0" />
         <geometry>
-          <cylinder radius="0.126" length="0.06" />
+          <cylinder radius="0.065" length="0.06" />
         </geometry>
       </collision>
@@ -77,5 +76,5 @@
       <parent link="chassis" />
       <child link="lidar_front" />
-      <origin rpy="0 0 0" xyz="0.26 0.43 0.01" />
+      <origin rpy="0 0 3.14159265359" xyz="0.26 0.43 0.01" />
     </joint>
     <link name="lidar_back">
@@ -115,5 +114,5 @@
         <origin rpy="0 1.57075 0" xyz="0 0 0" />
         <geometry>
-          <cylinder radius="0.126" length="0.06" />
+          <cylinder radius="0.065" length="0.06" />
         </geometry>
       </collision>
@@ -140,5 +139,5 @@
       <collision>
         <geometry>
-          <sphere radius="0.126" />
+          <sphere radius="0.065" />
         </geometry>
       </collision>
@@ -163,5 +162,5 @@
       <collision>
         <geometry>
-          <sphere radius="0.126" />
+          <sphere radius="0.065" />
         </geometry>
       </collision>
@@ -186,5 +185,5 @@
       <collision>
         <geometry>
-          <sphere radius="0.126" />
+          <sphere radius="0.065" />
         </geometry>
       </collision>
@@ -205,5 +204,5 @@
       <collision>
         <geometry>
-          <sphere radius="0.126" />
+          <sphere radius="0.065" />
         </geometry>
       </collision>
@@ -275,5 +274,5 @@
         <!-- kinematics -->
         <wheel_separation>0.62</wheel_separation>
-        <wheel_diameter>0.252</wheel_diameter>
+        <wheel_diameter>0.130</wheel_diameter>
         <!-- limits -->
         <max_wheel_torque>20</max_wheel_torque>
@@ -284,5 +283,5 @@
         <publish_wheel_tf>true</publish_wheel_tf>
         <odometry_frame>odom</odometry_frame>
-        <robot_base_frame>chassis</robot_base_frame>
+        <robot_base_frame>base_link</robot_base_frame>
       </plugin>
     </gazebo>
@@ -298,5 +297,5 @@
         <odom_topic>/odom</odom_topic>
         <odom_frame>odom</odom_frame>
-        <robot_base_frame>chassis</robot_base_frame>
+        <robot_base_frame>base_link</robot_base_frame>
         <tf_topic>/odom/tf</tf_topic>
       </plugin>

Commit message: fix: resolve git conflict marker in xacro file causing XML parser error

File: navigation/iros_mobile_platform_description/description/iros_mobile_platform_description.urdf.xacro (robot description, xacro)
@@ -185,9 +185,5 @@
       <collision>
         <geometry>
-<<<<<<< HEAD
-          <sphere radius="0.130" />
-=======
           <sphere radius="0.065" />
->>>>>>> dev_real
         </geometry>
       </collision>
