Commit message: fix: stabilize CAN initialization and correct base_link offset
- Added thread sleeps in motor driver node for reliable CAN startup
- Made CAN interface setup in hardware.launch.py more robust with sleeps and state checks
- Shifted chassis origin by +0.045m in X axis to align base_link with the physical rotation center

File: navigation/iros_mobile_platform_description/description/iros_mobile_platform_description.urdf.xacro (robot description, xacro)
@@ -6,5 +6,5 @@
       <parent link="base_link" />
       <child link="chassis" />
-      <origin rpy="0 0 -1.57079632679" xyz="0 0 0" />
+      <origin rpy="0 0 -1.57079632679" xyz="0.045 0 0" />
     </joint>
     <link name="chassis">

Commit message: refactor: Update wheel separation (track width) to 0.637m across all modules
- URDF Model: Increased `<wheel_separation>` to 0.637m in the diff-drive plugin and accurately shifted the left/right wheel joint origins (Y-axis from +/-0.31m to +/-0.3185m) to reflect the new physical dimensions.
- Controller Config: Updated `wheel_separation` parameter in `iros_mobile_platform_controllers.yaml` for correct odometry calculation.
- Controller Source: Changed the hardcoded default fallback value for `robot_base_` in `controller.cpp` to match the new 0.637m measurement.

File: navigation/iros_mobile_platform_description/description/iros_mobile_platform_description.urdf.xacro (robot description, xacro)
@@ -54,5 +54,5 @@
       <parent link="chassis" />
       <child link="left_wheel" />
-      <origin rpy="0 0 3.14" xyz="-0.31 -0.045 -0.15" />
+      <origin rpy="0 0 3.14" xyz="-0.3185 -0.045 -0.15" />
     </joint>
     <link name="lidar_front">
@@ -123,5 +123,5 @@
       <parent link="chassis" />
       <child link="right_wheel" />
-      <origin rpy="0 0 3.14" xyz="0.31 -0.045 -0.15" />
+      <origin rpy="0 0 3.14" xyz="0.3185 -0.045 -0.15" />
     </joint>
     <link name="front_left_dummy_wheel">
@@ -273,5 +273,5 @@
         <right_joint>chassis_to_right_wheel</right_joint>
         <!-- kinematics -->
-        <wheel_separation>0.62</wheel_separation>
+        <wheel_separation>0.637</wheel_separation>
         <wheel_diameter>0.130</wheel_diameter>
         <!-- limits -->
